File: quill-stm32wl.kicad_sch (KiCad schematic)
At the start: 32 parts, among them J1 USB_C_Receptacle_USB2.0_16P, J2 Conn_01x02_MountingPin, J3 Conn_01x12, J4 Conn_01x16, J5 Conn_01x04_MountingPin, J6 Conn_01x03_MountingPin, Q1 AO3401A, SW1 RESET, SW2 BOOT, U1 RAK3172-T-8-SM-I, U2 CH340E, U3 AP2112K-3.3, U4 MCP73831-2-OT

Commit message: assets, links, complete bom
Other:
- company: (none) -> Copyright (C) 2026 Olivér Pirger
Changed lines of the file:
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@@
 		(date "2026-05-07")
 		(rev "A")
+		(company "Copyright (C) 2026 Olivér Pirger")
 	)
 	(junction
